Commit message: 修复机械臂在 Gazebo 中漂浮漂移：新增 world→base_link 固定关节，删除无效的 fanuc_world

File: src/crx_description/urdf/crx10ia_l/crx10ia_l_macro.xacro (robot description, xacro)
@@ -12,4 +12,10 @@
     </material>
     <!-- links -->
+    <link name="world" />
+    <joint name="world_to_base" type="fixed">
+      <parent link="world"/>
+      <child link="base_link"/>
+      <origin xyz="0 0 0" rpy="0 0 0"/>
+    </joint>
     <link name="base_link">
       <visual>
@@ -209,11 +215,4 @@
       <limit lower="${-225 * pi / 180}" upper="${225 * pi / 180}" effort="0" velocity="${112 * pi / 180}"/>
     </joint>
-    <!-- fanuc world -->
-    <link name="fanuc_world" />
-    <joint name="base_link-fanuc_world" type="fixed">
-      <origin xyz="0 0 0.245" rpy="0 0 0"/>
-      <parent link="base_link"/>
-      <child link="fanuc_world"/>
-    </joint>
     <!-- flange -->
     <link name="flange" />
