Commit message: 接入 Robotiq 2F-85 夹爪仿真并修复控制与关节状态兼容问题

File: src/crx_control/urdf/crx10ia_l_gazebo.xacro (robot description, xacro)
@@ -4,4 +4,11 @@
   <xacro:include filename="$(find crx_control)/urdf/crx_gazebo.xacro"/>
   <xacro:crx10ia_l />
+  <!-- Anchor the pedestal while keeping all arm/gripper joints dynamic. -->
+  <link name="world"/>
+  <joint name="world_to_base" type="fixed">
+    <parent link="world"/>
+    <child link="base_link"/>
+    <origin xyz="0 0 0" rpy="0 0 0"/>
+  </joint>
   <xacro:crx_ros2_control_gazebo />
 </robot>

File: src/crx_control/urdf/crx_gazebo.xacro (robot description, xacro)
@@ -1,4 +1,5 @@
 <?xml version="1.0"?>
 <robot xmlns:xacro="http://www.ros.org/wiki/xacro">
+        <xacro:include filename="$(find crx_control)/urdf/robotiq_gazebo_control.xacro"/>
         <gazebo>
             <plugin filename="libgazebo_ros2_control.so" name="gazebo_ros2_control">
@@ -23,6 +24,6 @@
                 <joint name="J1">
                     <command_interface name="position">
-                        <param name="min">{-2*pi}</param>
-                        <param name="max">{2*pi}</param>
+                        <param name="min">${-2*pi}</param>
+                        <param name="max">${2*pi}</param>
                     </command_interface>
                     <command_interface name="effort">
@@ -37,6 +38,6 @@
                 <joint name="J2">
                     <command_interface name="position">
-                        <param name="min">{-2*pi}</param>
-                        <param name="max">{2*pi}</param>
+                        <param name="min">${-2*pi}</param>
+                        <param name="max">${2*pi}</param>
                     </command_interface>
                     <command_interface name="effort">
@@ -51,6 +52,6 @@
                 <joint name="J3">
                     <command_interface name="position">
-                        <param name="min">{-pi}</param>
-                        <param name="max">{pi}</param>
+                        <param name="min">${-pi}</param>
+                        <param name="max">${pi}</param>
                     </command_interface>
                     <command_interface name="effort">
@@ -65,6 +66,6 @@
                 <joint name="J4">
                     <command_interface name="position">
-                        <param name="min">{-2*pi}</param>
-                        <param name="max">{2*pi}</param>
+                        <param name="min">${-2*pi}</param>
+                        <param name="max">${2*pi}</param>
                     </command_interface>
                     <command_interface name="effort">
@@ -79,6 +80,6 @@
                 <joint name="J5">
                     <command_interface name="position">
-                        <param name="min">{-2*pi}</param>
-                        <param name="max">{2*pi}</param>
+                        <param name="min">${-2*pi}</param>
+                        <param name="max">${2*pi}</param>
                     </command_interface>
                     <command_interface name="effort">
@@ -93,6 +94,6 @@
                 <joint name="J6">
                     <command_interface name="position">
-                        <param name="min">{-2*pi}</param>
-                        <param name="max">{2*pi}</param>
+                        <param name="min">${-2*pi}</param>
+                        <param name="max">${2*pi}</param>
                     </command_interface>
                     <command_interface name="effort">
@@ -105,4 +106,5 @@
                     <state_interface name="velocity"/>
                 </joint>
+                <xacro:robotiq_gazebo_control/>
             </ros2_control>
         </xacro:macro>

File: src/crx_description/urdf/crx10ia_l/crx10ia_l_macro.xacro (robot description, xacro)
@@ -223,14 +223,26 @@
       <child link="flange" />
     </joint>
-    <!-- tcp -->
-    <link name="tcp" />
-    <joint name="flange-tcp" type="fixed">
+    <!-- Original tool orientation; camera stays on this mounting frame. -->
+    <link name="tool_mount" />
+    <joint name="flange-tool_mount" type="fixed">
       <origin xyz="0 0 0" rpy="0 ${pi/2} 0" />
       <parent link="flange" />
-      <child link="tcp" />
+      <child link="tool_mount" />
+    </joint>
+    <xacro:include filename="$(find crx_description)/urdf/gripper/robotiq_2f_85.xacro"/>
+    <xacro:robotiq_2f_85 prefix="" parent="tool_mount">
+      <origin xyz="0 0 0" rpy="0 0 0"/>
+    </xacro:robotiq_2f_85>
+    <!-- Nominal grasp reference, 145 mm along the gripper's approach axis.
+         This reference is fixed; actual fingertip height varies with opening. -->
+    <link name="tcp"/>
+    <joint name="gripper-tcp" type="fixed">
+      <parent link="robotiq_85_base_link"/>
+      <child link="tcp"/>
+      <origin xyz="0 0 0.145" rpy="0 0 0"/>
     </joint>
     <!-- ==================== 相机 ==================== -->
     <xacro:include filename="$(find crx_description)/urdf/camera/camera.xacro"/>
-    <xacro:camera_rgbd parent="tcp" name="camera">
+    <xacro:camera_rgbd parent="tool_mount" name="camera">
      <origin xyz="0 -0.08 0.02" rpy="0 -1.5708 0"/>
     </xacro:camera_rgbd>

File: src/crx_moveit_config/config/crx10ia_l.urdf.xacro (robot description, xacro)
@@ -1,9 +1,5 @@
 <?xml version="1.0"?>
 <robot xmlns:xacro="http://www.ros.org/wiki/xacro" name="crx10ia_l">
-    <xacro:arg name="initial_positions_file" default="$(find crx_control)/config/initial_positions.yaml" />
-    <!-- Import crx10ia_l urdf file -->
-    <xacro:include filename="$(find crx_description)/urdf/crx10ia_l/crx10ia_l.xacro" />
-    <!-- Import fake system ros2_control for MoveIt planning demo -->
-    <xacro:include filename="$(find crx_control)/urdf/crx10ia_l_fake_system.xacro" />
-    <xacro:crx10ia_l_ros2_control name="FakeSystem" initial_positions_file="$(arg initial_positions_file)"/>
+    <!-- Use exactly the same arm, gripper, TCP and control model as Gazebo. -->
+    <xacro:include filename="$(find crx_control)/urdf/crx10ia_l_gazebo.xacro"/>
 </robot>

Commit message: 修复底座穿透地面导致的 Gazebo 高频抖动

File: src/crx_control/urdf/crx10ia_l_gazebo.xacro (robot description, xacro)
@@ -9,5 +9,7 @@
     <parent link="world"/>
     <child link="base_link"/>
-    <origin xyz="0 0 0" rpy="0 0 0"/>
+    <!-- The base collision mesh extends 0.826 mm below its origin. Leave
+         clearance above the ground to avoid fighting the fixed constraint. -->
+    <origin xyz="0 0 0.002" rpy="0 0 0"/>
   </joint>
   <xacro:crx_ros2_control_gazebo />
